File: stm32_qfp64_breakout.sch (KiCad schematic (older format))
At the start: 25 parts, among them IC1 NCV8170, J1 Conn_01x24, J2 USB_HS, J3 USB_mini_micro_B, J4 Conn_01x24, J5 SWD, U2 STM32F205RGTx, Y1 8MHz Xtal

Commit message: pins are now 0.7 in apart
Parts:
- J1, J4: footprint Connector_PinHeader_2.54mm:PinHeader_1x24_P2.54mm_Vertical -> stm32_qfp64_breakout:M24_LOCK_NOSILK
Changed lines of the file:
@@
 F 0 "J1" H 1990 6220 50  0000 L CNN
 F 1 "Conn_01x24" H 1760 6140 50  0000 L CNN
-F 2 "Connector_PinHeader_2.54mm:PinHeader_1x24_P2.54mm_Vertical" H 2100 4900 50  0001 C CNN
+F 2 "stm32_qfp64_breakout:M24_LOCK_NOSILK" H 2100 4900 50  0001 C CNN
 F 3 "~" H 2100 4900 50  0001 C CNN
 	1    2100 4900
@@
 F 0 "J4" H 2718 3575 50  0000 C CNN
 F 1 "Conn_01x24" H 2718 3666 50  0000 C CNN
-F 2 "Connector_PinHeader_2.54mm:PinHeader_1x24_P2.54mm_Vertical" H 2800 5000 50  0001 C CNN
+F 2 "stm32_qfp64_breakout:M24_LOCK_NOSILK" H 2800 5000 50  0001 C CNN
 F 3 "~" H 2800 5000 50  0001 C CNN
 	1    2800 5000

Commit message: add microsd slot, refine layout
Parts:
- added D1: LED, flabbergast:LED-0603, symbol Device:LED
- added J6: Micro_SD_Card, stm32_qfp64_breakout:MOLEX_104031-0811, symbol stm32_qfp64_breakout:104031-0811
- added R2: 1kΩ, flabbergast:0603, symbol Device:R
- C1, C2: footprint Capacitor_SMD:C_0805_2012Metric -> Capacitor_SMD:C_0603_1608Metric
Connections:
- net GND: now also J1.23 (Pin_23), D1.1 (K), J6.6 (VSS), J6.9 (CARD_DET1), J6.G1 (GND), J6.G2 (GND), J6.G3 (GND), J6.G4 (GND); no longer J1.1 (Pin_1)
- net PA0: now also J1.8 (Pin_8); no longer J1.10 (Pin_10)
- net PA1: now also J1.9 (Pin_9); no longer J1.11 (Pin_11)
- net PA2: now also J1.10 (Pin_10); no longer J1.12 (Pin_12)
- net PA3: now also J1.11 (Pin_11); no longer J1.13 (Pin_13)
- net PA4: now also J1.12 (Pin_12); no longer J1.14 (Pin_14)
- net PA5: now also J1.13 (Pin_13); no longer J1.15 (Pin_15)
- net PA6: now also J1.14 (Pin_14); no longer J1.16 (Pin_16)
- net PA7: now also J1.15 (Pin_15); no longer J1.17 (Pin_17)
- net PB0: now also J1.18 (Pin_18); no longer J1.20 (Pin_20)
- net PB1: now also J1.19 (Pin_19); no longer J1.21 (Pin_21)
- net PB10: now also J1.21 (Pin_21); no longer J1.23 (Pin_23)
- net PB11: now also J1.22 (Pin_22); no longer J1.24 (Pin_24)
- net PB2: now also J1.20 (Pin_20); no longer J1.22 (Pin_22)
- net PB6: now also J6.10 (CARD_DET2)
- net PC0: now also J1.4 (Pin_4); no longer J1.6 (Pin_6)
- net PC1: now also J1.5 (Pin_5); no longer J1.7 (Pin_7)
- net PC10: now also J6.1 (DAT2)
- net PC11: now also J6.2 (CD/DAT3)
- net PC12: now also J6.5 (CLK)
- net PC13: now also J1.1 (Pin_1), R2.2; no longer J1.3 (Pin_3)
- net PC14: now also J1.2 (Pin_2); no longer J1.4 (Pin_4)
- net PC15: now also J1.3 (Pin_3); no longer J1.5 (Pin_5)
- net PC2: now also J1.6 (Pin_6); no longer J1.8 (Pin_8)
- net PC3: now also J1.7 (Pin_7); no longer J1.9 (Pin_9)
- net PC4: now also J1.16 (Pin_16); no longer J1.18 (Pin_18)
- net PC5: now also J1.17 (Pin_17); no longer J1.19 (Pin_19)
- net PC8: now also J6.7 (DAT0)
- net PC9: now also J6.8 (DAT1)
- net PD2: now also J6.3 (CMD)
- net VDD: now also J1.24 (Pin_24), J6.4 (VDD); no longer J1.2 (Pin_2)
- new net: D1.2 (A), R2.1
Changed lines of the file:
@@
 F 0 "C1" H 3775 1904 50  0000 R CNN
 F 1 "2.2µF" H 4010 2040 50  0000 R CNN
-F 2 "Capacitor_SMD:C_0805_2012Metric" H 3928 1800 50  0001 C CNN
+F 2 "Capacitor_SMD:C_0603_1608Metric" H 3928 1800 50  0001 C CNN
 F 3 "~" H 3890 1950 50  0001 C CNN
 	1    3890 1950
@@
 F 0 "C2" H 4315 2096 50  0000 L CNN
 F 1 "2.2µF" H 4315 2005 50  0000 L CNN
-F 2 "Capacitor_SMD:C_0805_2012Metric" H 4238 1900 50  0001 C CNN
+F 2 "Capacitor_SMD:C_0603_1608Metric" H 4238 1900 50  0001 C CNN
 F 3 "~" H 4200 2050 50  0001 C CNN
 	1    4200 2050
@@
 NoConn ~ 5100 1200
 Wire Wire Line
+	1900 4100 1800 4100
+Wire Wire Line
+	1900 4200 1800 4200
+Wire Wire Line
 	1900 4300 1800 4300
 Wire Wire Line
@@
 Wire Wire Line
 	1900 4600 1800 4600
-Wire Wire Line
-	1900 4700 1800 4700
-Wire Wire Line
-	1900 4800 1800 4800
+Text GLabel 1800 4100 0    50   Output ~ 0
+PC0
+Text GLabel 1800 4200 0    50   Output ~ 0
+PC1
 Text GLabel 1800 4300 0    50   Output ~ 0
-PC0
+PC2
 Text GLabel 1800 4400 0    50   Output ~ 0
-PC1
+PC3
+Text GLabel 1800 5300 0    50   Output ~ 0
+PC4
+Text GLabel 1800 5400 0    50   Output ~ 0
+PC5
+Wire Wire Line
+	1800 5400 1900 5400
+Wire Wire Line
+	1800 5300 1900 5300
+Wire Wire Line
+	1800 5200 1900 5200
+Wire Wire Line
+	1800 5100 1900 5100
+Wire Wire Line
+	1800 5000 1900 5000
+Wire Wire Line
+	1800 4900 1900 4900
+Wire Wire Line
+	1800 4800 1900 4800
+Wire Wire Line
+	1800 4700 1900 4700
 Text GLabel 1800 4500 0    50   Output ~ 0
-PC2
+PA0
 Text GLabel 1800 4600 0    50   Output ~ 0
-PC3
+PA1
+Text GLabel 1800 4700 0    50   Output ~ 0
+PA2
+Text GLabel 1800 4800 0    50   Output ~ 0
+PA3
+Text GLabel 1800 4900 0    50   Output ~ 0
+PA4
+Text GLabel 1800 5000 0    50   Output ~ 0
+PA5
+Text GLabel 1800 5100 0    50   Output ~ 0
+PA6
+Text GLabel 1800 5200 0    50   Output ~ 0
+PA7
+Wire Wire Line
+	1800 5600 1900 5600
+Wire Wire Line
+	1800 5500 1900 5500
 Text GLabel 1800 5500 0    50   Output ~ 0
-PC4
-Text GLabel 1800 5600 0    50   Output ~ 0
-PC5
-Wire Wire Line
-	1800 5600 1900 5600
-Wire Wire Line
-	1800 5500 1900 5500
-Wire Wire Line
-	1800 5400 1900 5400
-Wire Wire Line
-	1800 5300 1900 5300
-Wire Wire Line
-	1800 5200 1900 5200
-Wire Wire Line
-	1800 5100 1900 5100
-Wire Wire Line
-	1800 5000 1900 5000
-Wire Wire Line
-	1800 4900 1900 4900
-Text GLabel 1800 4700 0    50   Output ~ 0
-PA0
-Text GLabel 1800 4800 0    50   Output ~ 0
-PA1
-Text GLabel 1800 4900 0    50   Output ~ 0
-PA2
-Text GLabel 1800 5000 0    50   Output ~ 0
-PA3
-Text GLabel 1800 5100 0    50   Output ~ 0
-PA4
-Text GLabel 1800 5200 0    50   Output ~ 0
-PA5
-Text GLabel 1800 5300 0    50   Output ~ 0
-PA6
-Text GLabel 1800 5400 0    50   Output ~ 0
-PA7
+PB0
+Wire Wire Line
+	1800 5900 1900 5900
 Wire Wire Line
 	1800 5800 1900 5800
-Wire Wire Line
-	1800 5700 1900 5700
-Text GLabel 1800 5700 0    50   Output ~ 0
-PB0
-Wire Wire Line
-	1800 6100 1900 6100
-Wire Wire Line
-	1800 6000 1900 6000
-Text GLabel 1800 6000 0    50   Output ~ 0
+Text GLabel 1800 5800 0    50   Output ~ 0
 PB10
-Text GLabel 1800 6100 0    50   Output ~ 0
+Text GLabel 1800 5900 0    50   Output ~ 0
 PB11
 Wire Wire Line
+	1900 3800 1800 3800
+Wire Wire Line
+	1900 3900 1800 3900
+Wire Wire Line
 	1900 4000 1800 4000
-Wire Wire Line
-	1900 4100 1800 4100
-Wire Wire Line
-	1900 4200 1800 4200
+Text GLabel 1800 3800 0    50   Output ~ 0
+PC13
+Text GLabel 1800 3900 0    50   Output ~ 0
+PC14
 Text GLabel 1800 4000 0    50   Output ~ 0
-PC13
-Text GLabel 1800 4100 0    50   Output ~ 0
-PC14
-Text GLabel 1800 4200 0    50   Output ~ 0
 PC15
 Wire Wire Line
@@
 	8240 1200 8580 1200
 Connection ~ 8580 1200
-Text GLabel 1800 5800 0    50   Output ~ 0
+Text GLabel 1800 5600 0    50   Output ~ 0
 PB1
 Wire Wire Line
@@
 Text GLabel 6100 3300 2    50   Output ~ 0
 PB2
-Text GLabel 1800 5900 0    50   Output ~ 0
+Text GLabel 1800 5700 0    50   Output ~ 0
 PB2
 Wire Wire Line
-	1800 5900 1900 5900
+	1800 5700 1900 5700
 Text GLabel 3100 3900 2    50   Output ~ 0
 PB8
@@
 Text GLabel 3730 6570 2    50   Output ~ 0
 SWCLK
-Text GLabel 1800 3800 0    50   Output ~ 0
+Text GLabel 1800 6000 0    50   Output ~ 0
 GND
-Text GLabel 1800 3900 0    50   Output ~ 0
+Text GLabel 1800 6100 0    50   Output ~ 0
 VDD
 Wire Wire Line
-	1900 3900 1800 3900
-Wire Wire Line
-	1900 3800 1800 3800
+	1900 6100 1800 6100
+Wire Wire Line
+	1900 6000 1800 6000
 Wire Wire Line
 	3640 6570 3730 6570
@@
 Wire Wire Line
 	2800 1700 3100 1700
+Wire Wire Line
+	8300 4750 8200 4750
+Wire Wire Line
+	8300 4850 8200 4850
+Wire Wire Line
+	8300 4950 8200 4950
+Wire Wire Line
+	8300 5550 8200 5550
+Wire Wire Line
+	8300 5050 8200 5050
+Wire Wire Line
+	8300 4550 8200 4550
+Wire Wire Line
+	8300 4650 8200 4650
+Text GLabel 8200 4750 0    50   Output ~ 0
+PC10
+Text GLabel 8200 4850 0    50   Output ~ 0
+PC11
+Text GLabel 8200 5550 0    50   Output ~ 0
+VDD
+Text GLabel 8200 5050 0    50   Output ~ 0
+PC12
+Text GLabel 8200 4550 0    50   Output ~ 0
+PC8
+Text GLabel 8200 4650 0    50   Output ~ 0
+PC9
+Text GLabel 8200 4950 0    50   Output ~ 0
+PD2
+Text GLabel 8200 5650 0    50   Output ~ 0
+GND
+Wire Wire Line
+	8300 5650 8200 5650
+Text GLabel 9400 5600 2    50   Output ~ 0
+GND
+Wire Wire Line
+	9300 5600 9400 5600
+Wire Wire Line
+	8300 5350 8200 5350
+$Comp
+L stm32_qfp64_breakout:104031-0811 J6
+U 1 1 5EFB2915
+P 8800 5100
+F 0 "J6" H 8800 5867 50  0000 C CNN
+F 1 "Micro_SD_Card" H 8800 5776 50  0000 C CNN
+F 2 "stm32_qfp64_breakout:MOLEX_104031-0811" H 9950 5400 50  0001 C CNN
+F 3 "" H 8800 5100 50  0001 C CNN
+	1    8800 5100
+	1    0    0    -1
+$EndComp
+Wire Wire Line
+	8300 5250 8200 5250
+Text GLabel 8200 5250 0    50   Output ~ 0
+GND
+Text GLabel 8200 5350 0    50   Output ~ 0
+PB6
+$Comp
+L Device:LED D1
+U 1 1 5F30A693
+P 6800 5550
+F 0 "D1" V 6747 5628 50  0000 L CNN
+F 1 "LED" V 6838 5628 50  0000 L CNN
+F 2 "flabbergast:LED-0603" H 6800 5550 50  0001 C CNN
+F 3 "~" H 6800 5550 50  0001 C CNN
+	1    6800 5550
+	0    -1   -1   0
+$EndComp
+Wire Wire Line
+	6800 5700 6800 5800
+$Comp
+L power:GND #PWR01
+U 1 1 5F354908
+P 6800 5800
+F 0 "#PWR01" H 6800 5550 50  0001 C CNN
+F 1 "GND" H 6805 5627 50  0000 C CNN
+F 2 "" H 6800 5800 50  0001 C CNN
+F 3 "" H 6800 5800 50  0001 C CNN
+	1    6800 5800
+	1    0    0    -1
+$EndComp
+Wire Wire Line
+	6800 5400 6800 5300
+$Comp
+L Device:R R2
+U 1 1 5F365C36
+P 6650 5300
+F 0 "R2" V 6443 5300 50  0000 C CNN
+F 1 "1kΩ" V 6534 5300 50  0000 C CNN
+F 2 "flabbergast:0603" V 6580 5300 50  0001 C CNN
+F 3 "~" H 6650 5300 50  0001 C CNN
+	1    6650 5300
+	0    1    1    0
+$EndComp
+Wire Wire Line
+	6500 5300 6400 5300
+Text GLabel 6400 5300 0    50   Output ~ 0
+PC13
 $EndSCHEMATC
